File: Hardware/KiCad-V2/denise-adapter.kicad_pcb (KiCad board)
At the start: 2 copper layers, 51.5 x 72.5 mm, 15 parts, among them J1 Conn_02x20_Odd_Even, J2 Conn_01x04, J3 Conn_01x04, J4 Conn_01x04, U1 Denise, U2 Denise, U3 SN74CBTD16211, U4 SN74CBTD16211, U5 TPS73643DBV

Commit message: Should use SN74CBT16211A, not SN74CBTD16211
Parts:
- U3, U4: value SN74CBTD16211 -> SN74CBT16211A
Changed lines of the file:
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@@
       (effects (font (size 1 1) (thickness 0.15)))
     )
-    (fp_text value SN74CBTD16211 (at 0 8.05) (layer F.Fab)
+    (fp_text value SN74CBT16211A (at 0 8.05) (layer F.Fab)
       (effects (font (size 1 1) (thickness 0.15)))
     )
@@
       (effects (font (size 1 1) (thickness 0.15)))
     )
-    (fp_text value SN74CBTD16211 (at 0 8.05) (layer F.Fab)
+    (fp_text value SN74CBT16211A (at 0 8.05) (layer F.Fab)
       (effects (font (size 1 1) (thickness 0.15)))
     )

Commit message: Fixed label +4V to correct value +4V3
Connections:
- net +4V renamed +4V3
Changed lines of the file:
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@@
   (net 104 "Net-(U4-Pad27)")
   (net 105 "Net-(JP1-Pad2)")
-  (net 106 +4V)
+  (net 106 +4V3)
   (net 107 "Net-(U5-Pad4)")
   (net_class Default "This is the default net class."
@@
     (uvia_drill 0.1)
     (add_net +3V3)
-    (add_net +4V)
+    (add_net +4V3)
     (add_net +5V)
     (add_net 3VB0)
@@
     )
     (pad 5 smd rect (at 1.1 -0.95 180) (size 1.06 0.65) (layers F.Cu F.Paste F.Mask)
-      (net 106 +4V))
+      (net 106 +4V3))
     (pad 4 smd rect (at 1.1 0.95 180) (size 1.06 0.65) (layers F.Cu F.Paste F.Mask)
       (net 107 "Net-(U5-Pad4)"))
@@
       (net 35 3VZD))
     (pad 17 smd rect (at -3.75 1.25 180) (size 1 0.285) (layers F.Cu F.Paste F.Mask)
-      (net 106 +4V))
+      (net 106 +4V3))
     (pad 16 smd rect (at -3.75 0.75 180) (size 1 0.285) (layers F.Cu F.Paste F.Mask)
       (net 33 3VCSYNC))
@@
       (net 15 3VD10))
     (pad 17 smd rect (at -3.75 1.25 180) (size 1 0.285) (layers F.Cu F.Paste F.Mask)
-      (net 106 +4V))
+      (net 106 +4V3))
     (pad 16 smd rect (at -3.75 0.75 180) (size 1 0.285) (layers F.Cu F.Paste F.Mask)
       (net 12 3VD0))
@@
       (net 1 GND))
     (pad 1 smd roundrect (at -1.4875 0 270) (size 1.425 1.75) (layers B.Cu B.Paste B.Mask) (roundrect_rratio 0.175439)
-      (net 106 +4V))
+      (net 106 +4V3))
     (model ${KISYS3DMOD}/Capacitor_SMD.3dshapes/C_1206_3216Metric.wrl
       (at (xyz 0 0 0))
@@
       (net 1 GND))
     (pad 1 smd roundrect (at -1.4875 0 90) (size 1.425 1.75) (layers B.Cu B.Paste B.Mask) (roundrect_rratio 0.175439)
-      (net 106 +4V))
+      (net 106 +4V3))
     (model ${KISYS3DMOD}/Capacitor_SMD.3dshapes/C_1206_3216Metric.wrl
       (at (xyz 0 0 0))
